File: hardware/chainclock.brd (EAGLE design)
At the start: 40 x 50 mm, 28 parts, among them IC1 TINY2313-*S*, Q1 IRLML2502, Q2 IRLML2502, Q3 IRLML2502, Q4 IRLML2502, Q6 BSS84, Y1 8MHz

Commit message: voltage divider resistor values fixed
Parts:
- R6: value 100 -> 5k6
- R7: value 100 -> 10k
Changed lines of the file:
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@@
 <attribute name="VALUE" x="14.097" y="38.7985" size="1.27" layer="27" rot="R90"/>
 </element>
-<element name="R6" library="resistor" package="R0603" value="100" x="30.7975" y="42.8625" smashed="yes" rot="R270">
+<element name="R6" library="resistor" package="R0603" value="5k6" x="30.7975" y="42.8625" smashed="yes" rot="R270">
 <attribute name="NAME" x="31.4325" y="44.7675" size="1.27" layer="25" font="vector" rot="R90"/>
 <attribute name="VALUE" x="28.7655" y="43.7515" size="1.27" layer="27" rot="R270"/>
 </element>
-<element name="R7" library="resistor" package="R0603" value="100" x="27.94" y="39.6875" smashed="yes" rot="R270">
+<element name="R7" library="resistor" package="R0603" value="10k" x="27.94" y="39.6875" smashed="yes" rot="R270">
 <attribute name="NAME" x="30.1625" y="39.37" size="1.27" layer="25" font="vector" rot="R90"/>
 <attribute name="VALUE" x="25.908" y="40.5765" size="1.27" layer="27" rot="R270"/>
